File: PCD.brd (EAGLE design)
At the start: 64 x 56 mm, 23 parts, among them IC2 TCAN332DR, IC4 MCP2515, J1 M40-SOCKET-BELOW, J2 DC IN, J4 DC IN, J5 CAN Termination

Commit message: Added nets for HAT EEPROM
Connections:
- new net ID_SC: J1.28
- new net ID_SD: J1.27
Changed lines of the file:
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@@
 <wire x1="61.222" y1="24.54" x2="62" y2="23.762" width="0.254" layer="1"/>
+</signal>
+<signal name="ID_SD">
+<contactref element="J1" pad="27"/>
+</signal>
+<signal name="ID_SC">
+<contactref element="J1" pad="28"/>
 </signal>
 </signals>

Commit message: Major work for v1.0 release
Parts:
- removed R17: 10K, SuperHouse-DiscreteSemi:R0603
- removed R6: 120R, SuperHouse-DiscreteSemi:R0603
- added R2: 120R, SuperHouse-DiscreteSemi:R0603
- added R3: 10K, SuperHouse-DiscreteSemi:R0603
- added SJ3: (no value), freetronics-jon:SJ
- J3: value (none) -> PoE IN
- J6: value CAN -> CAN_1
- J7: value CAN -> CAN_2
- moved IC2 2.54 mm to (50.0, 11.5)
- renumbered IC4 to IC1, JP1 to J6, JP2 to J7, R8 to R4, R9 to R1
Connections:
- new net CAN_PWR: J6.1, J7.1, SJ3.1
- net CANH: now also R2.1; no longer R6.1
- net GND: now also R3.1; no longer R17.1
- net N$26: now also R3.2; no longer R17.2
- net N$3: now also R2.2; no longer R6.2
- net POS: now also SJ3.2; no longer J6.1, J7.1
Routing:
- net POS: track 91.2 -> 82.1 mm
- net CAN_PWR: track 0.00 -> 8.15 mm
- net N$29: track 15.8 -> 18.0 mm
- net 3.3V: track 80.0 -> 77.9 mm
- net N$28: track 4.87 -> 6.83 mm
- net CANH: track 15.6 -> 16.7 mm
- net N$3: track 3.32 -> 4.03 mm
- net N$26: track 4.25 -> 4.79 mm
Other:
- board text added: "3.3V"
- board text added: "A"
- board text added: "CAN Term"
- board text added: "K"
- board text added: "SCL"
- board text added: "SDA"
