File: PCD.sch (EAGLE design)
At the start: 15 parts, among them J1 M40-SOCKET-BELOW, J2 DC IN, J4 DC IN, J5 OLED, J7 M14PTH, J8 M06-PLAIN, J9 M06-PLAIN

Commit message: Basic schematic and routing. Time to ponder it for a while.
Parts:
- removed J7: M14PTH, freetronics-jon:M14PTH
- removed J8, J9: M06-PLAIN, SuperHouse-Connectors:M06-PLAIN
- added C13, C14: 15pF, SuperHouse-DiscreteSemi:CAP0603
- added IC2: TCAN332DR, SuperHouse-ICs:MCP2551
- added IC4: MCP2515, SuperHouse-ICs:MCP2515
- added JP1, JP2: CAN, SuperHouse-Connectors:M04-PIN
- added MOD1: OLED-I2C128X64-0.96, SuperHouse-Displays:OLED-I2C128X64-0.96
- added R17, R9: 10K, SuperHouse-DiscreteSemi:RESISTOR0603
- added R6: 120R, SuperHouse-DiscreteSemi:RESISTOR0603
- added XTL3: 16MHz, SuperHouse-Oscillators:CRYSTAL-GND3X2
- J5: value OLED -> CAN Termination; device SuperHouse-Connectors:M04-PLAIN -> SuperHouse-Connectors:M02-PIN
Connections:
- new net CANH: IC2.CANH, JP1.2, JP2.2, R6.1
- new net CANL: IC2.CANL, J5.1, JP1.3, JP2.3
- new net IO12: IC4.!INT, J1.32
- new net IO8: IC4.!CS, J1.24
- new net MISO: IC4.SO, J1.21
- new net MOSI: IC4.SI, J1.19
- new net N$26: IC2.RS, R17.2
- new net N$28: IC2.TXD, IC4.TXCAN
- new net N$29: IC2.RXD, IC4.RXCAN
- new net N$3: J5.2, R6.2
- new net N$30: C13.2, IC4.OSC1, XTL3.XTL2
- new net N$48: C14.2, IC4.OSC2, XTL3.XTL1
- new net N$49: IC4.!RST, R9.1
- new net SCK: IC4.SCK, J1.23
- net 3.3V: now also IC2.VDD, IC4.VDD, MOD1.VCC, R9.2; no longer J5.3, J9.1, J9.2, J9.3, J9.4, J9.5, J9.6
- net 5V: no longer J8.1, J8.2, J8.3, J8.4, J8.5, J8.6
- net GND: now also C13.1, C14.1, IC2.VSS, IC4.VSS, JP1.4, JP2.4, MOD1.GND, R17.1, XTL3.GND, XTL3.GND2; no longer J5.4, J7.1, J7.10, J7.11, J7.12, J7.13, J7.14, J7.2, J7.3, J7.4, J7.5, J7.6, J7.7, J7.8, J7.9
- net POS: now also JP1.1, JP2.1
- net SCL: now also MOD1.SCL; no longer J5.2
- net SDA: now also MOD1.SDA; no longer J5.1
Other:
- note added: "0.96" I2C OLED"
- note added: "CAN Bus Hat for Raspberry Pi"
- note added: "CAN Bus Interface"
- note added: "Note: TCAN332DR is used instead of MCP2551 because it can operate at 3.3V"
- note added: "SKU: PICANDISPLAY"
- note removed: "I2C OLED Header"
- note removed: "Power Rails"
- note removed: "Prototyping Area"
- note removed: "SKU: VOLTHAT"
- note removed: "VoltHat PoE Voltage Regulator for Raspberry Pi"

Commit message: Added nets for HAT EEPROM
Connections:
- new net ID_SC: J1.28
- new net ID_SD: J1.27
Changed lines of the file:
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@@
+</segment>
+</net>
+<net name="ID_SD" class="0">
+<segment>
+<pinref part="J1" gate="G$1" pin="27"/>
+<wire x1="22.86" y1="134.62" x2="17.78" y2="134.62" width="0.1524" layer="91"/>
+<label x="17.78" y="134.62" size="1.27" layer="95" rot="R180" xref="yes"/>
+</segment>
+</net>
+<net name="ID_SC" class="0">
+<segment>
+<pinref part="J1" gate="G$1" pin="28"/>
+<wire x1="38.1" y1="134.62" x2="43.18" y2="134.62" width="0.1524" layer="91"/>
+<label x="43.18" y="134.62" size="1.27" layer="95" xref="yes"/>
 </segment>
 </net>

Commit message: Major work for v1.0 release
Parts:
- removed IC4: MCP2515, SuperHouse-ICs:MCP2515
- removed JP1, JP2: CAN, SuperHouse-Connectors:M04-PIN
- removed R17, R9: 10K, SuperHouse-DiscreteSemi:RESISTOR0603
- removed R6: 120R, SuperHouse-DiscreteSemi:RESISTOR0603
- removed R8: 2K2, SuperHouse-DiscreteSemi:RESISTOR0603
- added IC1: MCP2515, SuperHouse-ICs:MCP2515
- added J6: CAN_1, SuperHouse-Connectors:M04-PIN
- added J7: CAN_2, SuperHouse-Connectors:M04-PIN
- added R1, R3: 10K, SuperHouse-DiscreteSemi:RESISTOR0603
- added R2: 120R, SuperHouse-DiscreteSemi:RESISTOR0603
- added R4: 2K2, SuperHouse-DiscreteSemi:RESISTOR0603
- added SJ3: (no value), freetronics-jon:SJN
- J3: value (none) -> PoE IN
Connections:
- new net CAN_PWR: J6.1, J7.1, SJ3.1
- net 3.3V: now also IC1.VDD, R1.2; no longer IC4.VDD, R9.2
- net 5V: now also R4.1; no longer R8.1
- net CANH: now also J6.2, J7.2, R2.1; no longer JP1.2, JP2.2, R6.1
- net CANL: now also J6.3, J7.3; no longer JP1.3, JP2.3
- net GND: now also IC1.VSS, J6.4, J7.4, R3.1; no longer IC4.VSS, JP1.4, JP2.4, R17.1
- net IO12: now also IC1.!INT; no longer IC4.!INT
- net IO8: now also IC1.!CS; no longer IC4.!CS
- net MISO: now also IC1.SO; no longer IC4.SO
- net MOSI: now also IC1.SI; no longer IC4.SI
- net N$203: now also R4.2; no longer R8.2
- net N$26: now also R3.2; no longer R17.2
- net N$28: now also IC1.TXCAN; no longer IC4.TXCAN
- net N$29: now also IC1.RXCAN; no longer IC4.RXCAN
- net N$3: now also R2.2; no longer R6.2
- net N$30: now also IC1.OSC1; no longer IC4.OSC1
- net N$48: now also IC1.OSC2; no longer IC4.OSC2
- net N$49: now also IC1.!RST, R1.1; no longer IC4.!RST, R9.1
- net POS: now also SJ3.2; no longer JP1.1, JP2.1
- net SCK: now also IC1.SCK; no longer IC4.SCK
Other:
- note added: "Note: - Solder across jumpers SJ1 and SJ2 to receive power via PoE - Solder across jumper SJ3 to receive or deliver power to CAN"
- note added: "Raspberry Pi CAN Bus Display"
- note added: "SKU: PCD"
- note added: "v1.0 (2019-11-27)"
- note added: "www.superhouse.tv/pcd"
- note removed: "CAN Bus Hat for Raspberry Pi"
- note removed: "Note: Solder across jumpers SJ1 and SJ2 to receive power via PoE"
- note removed: "SKU: PICANDISPLAY"
- note removed: "v2.0 (2019-07-01)"
- note removed: "www.superhouse.tv/volthat"
- moved on the sheet: C13, C14, D1, D2, IC2, J1, J2, J3, J4, J5, LED3, MOD1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
